Commit message: feat: add floating claptrap simulation setup
Retopologize the URDF around the intended robot semantics: base_link is the structure reference, plane1 and plane2 are fixed frame plates, link1 is the walking wheel, and link2 is the momentum wheel.

Add a generated floating MJCF variant and scene entry that include a root freejoint, so gravity can move the robot and fall-over behavior can be tested in MuJoCo.

Add smaller actuator control ranges for the walking wheel and momentum wheel, and extend the MJCF update script to regenerate and validate fixed, floating, and scene XML outputs without compile overwrite prompts.

File: model/urdf/claptrap.urdf (robot description, URDF)
Before this commit: robot claptrap, 6 links, 5 joints
Links:
- link base_link: mass 0.0001 -> None; geometry 
Joints:
- removed joint link1_to_plane1
- added joint base_link_to_plane1: type fixed, parent base_link, child plane1, origin xyz=0 0.1 0 rpy=0 0 0
- joint base_link_to_link1: limit lower=-1 upper=1 effort=1000.0 velocity=0.5 -> effort=1000.0 velocity=30; origin xyz=0 0 3.0814879110195774e-33 rpy=0 0 -2.4651903288156613e-32 -> xyz=0 0 0 rpy=0 0 0; type revolute -> continuous
- joint plane1_to_link2: limit lower=-1 upper=1 effort=1000.0 velocity=0.5 -> effort=1000.0 velocity=100; type revolute -> continuous
- joint plane1_to_plane2: origin xyz=4.9303806576313234e-33 0.12 0 rpy=6.07716335728627e-64 0 1.4981364335015033e-95 -> xyz=0 0.12 0 rpy=0 0 0

Commit message: feat: add imu markers and sensors
Add four fixed IMU marker links on plane1 so the URDF exposes physical sensor locations at the frame corners.

Keep fixed URDF bodies in generated MJCF by disabling fusestatic, allowing MuJoCo XML body names to stay aligned with the URDF topology.

Add MuJoCo frame-based IMU sensor outputs for orientation, angular velocity, and linear acceleration, and keep the updated wheel actuator control ranges.

File: model/urdf/claptrap.urdf (robot description, URDF)
Before this commit: robot claptrap, 6 links, 5 joints
Links:
- added link imu_front_left, mass 0.005; collision box size=0.015 0.008 0.015; visual box size=0.015 0.008 0.015
- added link imu_front_right, mass 0.005; collision box size=0.015 0.008 0.015; visual box size=0.015 0.008 0.015
- added link imu_rear_left, mass 0.005; collision box size=0.015 0.008 0.015; visual box size=0.015 0.008 0.015
- added link imu_rear_right, mass 0.005; collision box size=0.015 0.008 0.015; visual box size=0.015 0.008 0.015
Joints:
- added joint plane1_to_imu_front_left: type fixed, parent plane1, child imu_front_left, origin xyz=0.06 0.008 0.06 rpy=0 0 0
- added joint plane1_to_imu_front_right: type fixed, parent plane1, child imu_front_right, origin xyz=0.06 0.008 -0.06 rpy=0 0 0
- added joint plane1_to_imu_rear_left: type fixed, parent plane1, child imu_rear_left, origin xyz=-0.06 0.008 0.06 rpy=0 0 0
- added joint plane1_to_imu_rear_right: type fixed, parent plane1, child imu_rear_right, origin xyz=-0.06 0.008 -0.06 rpy=0 0 0

Commit message: feat: update imu marker layout

File: model/urdf/claptrap.urdf (robot description, URDF)
Before this commit: robot claptrap, 10 links, 9 joints
Links:
- removed link imu_front_left
- removed link imu_front_right
- removed link imu_rear_left
- removed link imu_rear_right
- added link imu_plane1_diag_a, mass 0.005; collision box size=0.015 0.008 0.015; visual box size=0.015 0.008 0.015
- added link imu_plane1_diag_b, mass 0.005; collision box size=0.015 0.008 0.015; visual box size=0.015 0.008 0.015
- added link imu_plane2_diag_a, mass 0.005; collision box size=0.015 0.008 0.015; visual box size=0.015 0.008 0.015
- added link imu_plane2_diag_b, mass 0.005; collision box size=0.015 0.008 0.015; visual box size=0.015 0.008 0.015
Joints:
- removed joint plane1_to_imu_front_left
- removed joint plane1_to_imu_front_right
- removed joint plane1_to_imu_rear_left
- removed joint plane1_to_imu_rear_right
- added joint plane1_to_imu_diag_a: type fixed, parent plane1, child imu_plane1_diag_a, origin xyz=0.06 0.008 0.06 rpy=0 0 0
- added joint plane1_to_imu_diag_b: type fixed, parent plane1, child imu_plane1_diag_b, origin xyz=-0.06 0.008 -0.06 rpy=0 0 0
- added joint plane2_to_imu_diag_a: type fixed, parent plane2, child imu_plane2_diag_a, origin xyz=0.075 0.008 0.075 rpy=0 0 0
- added joint plane2_to_imu_diag_b: type fixed, parent plane2, child imu_plane2_diag_b, origin xyz=-0.075 0.008 -0.075 rpy=0 0 0

Commit message: Update URDF frames and estimator attitude rates

File: model/urdf/claptrap.urdf (robot description, URDF)
Before this commit: robot claptrap, 10 links, 9 joints
Joints:
- joint base_joint: origin xyz=0 0 0.1 rpy=1.5707963267948963 0 0 -> xyz=0 0 0.1 rpy=0 0 0
- joint base_link_to_link1: limit effort=1000.0 velocity=30 -> effort=1000 velocity=30; origin xyz=0 0 0 rpy=0 0 0 -> xyz=0 0 0 rpy=1.5707963 0 0
- joint base_link_to_plane1: origin xyz=0 0.1 0 rpy=0 0 0 -> xyz=0 0 0.1 rpy=0 0 0
- joint plane1_to_imu_diag_a: origin xyz=0.06 0.008 0.06 rpy=0 0 0 -> xyz=0.065 0.065 0.008 rpy=0 0 0
- joint plane1_to_imu_diag_b: origin xyz=-0.06 0.008 -0.06 rpy=0 0 0 -> xyz=-0.065 -0.065 0.008 rpy=0 0 0
- joint plane1_to_link2: limit effort=1000.0 velocity=100 -> effort=1000 velocity=100; origin xyz=0 0.06 0 rpy=2.0344439357957027 -1.5707963267948966 1.1071487177940904 -> xyz=0 0 0.06 rpy=2.0344439 -1.5707963 1.1071487
- joint plane1_to_plane2: origin xyz=0 0.12 0 rpy=0 0 0 -> xyz=0 0 0.12 rpy=0 0 0
- joint plane2_to_imu_diag_a: origin xyz=0.075 0.008 0.075 rpy=0 0 0 -> xyz=0.08 0.08 0.008 rpy=0 0 0
- joint plane2_to_imu_diag_b: origin xyz=-0.075 0.008 -0.075 rpy=0 0 0 -> xyz=-0.08 -0.08 0.008 rpy=0 0 0
